Commit message: revise some files

File: urdf_tutorials/urdf/joints.urdf (robot description, URDF)
Before this commit: robot joint_origins, 3 links, 2 joints
Joints:
- removed joint first_arm_to_second_arm
- added joint first_base_to_second_arm: type revolute, parent base_link, child second_arm, origin xyz=0 0.22 0.25 rpy=0 0 0, axis 0 1 0, limit lower=-1.57 upper=1.57 effort=20 velocity=10
- joint base_to_first_arm: axis (none) -> 0 1 0; limit (none) -> lower=-1.57 upper=1.57 effort=20 velocity=10; origin xyz=0 -0.22 0.25 -> xyz=0 -0.22 0.25 rpy=0 0 0; type fixed -> revolute
